File: ModuleV440/ModuleV440.kicad_pcb (KiCad board)
At the start: 2 copper layers, 30 x 61.3 mm, 45 parts, among them J2 AVR-ISP-6, Q1 AO3400A, U1 EL3H7(B)(TA)-G, Y1 8MHZ Ceramic Resonator

Commit message: prismatic diyBMS boards for LF230 / LF280 cells
Parts:
- removed R12, R22, R24, R25, R26, R29, R6, R8: 3.3OHM 3/4W, Resistor_SMD:R_2010_5025Metric
- R30: footprint Resistor_SMD:R_2010_5025Metric -> Resistor_THT:R_Radial_Power_L13.0mm_W9.0mm_P5.00mm
- moved R30 11.5 mm to (114.6, 87.1)
Connections:
- R30 pad 1: Net-(R26-Pad2) -> VCC
Routing:
- net Net-(Q1-D): track 37.9 -> 13.1 mm
- net VCC: track 132.0 -> 123.6 mm
- net Net-(R24-Pad2): track 5.60 -> 0.00 mm
- net Net-(R22-Pad2): track 5.59 -> 0.00 mm
- net Net-(R6-Pad2): track 5.58 -> 0.00 mm
- net Net-(R25-Pad2): track 5.58 -> 0.00 mm
- net Net-(R12-Pad1): track 5.58 -> 0.00 mm
- net Net-(R26-Pad2): track 5.53 -> 0.00 mm
- net Net-(Q1-G): track 48.1 -> 50.4 mm
Other:
- net class Default removed
- net class Power removed
- board text removed: "DANGER HOT!"
- board text removed: "JLCJLCJLCJLC"
- board text removed: "©2019-2021 Stuart Pittaway"
